Commit message: Add files via upload

File: Practica1/urdf_models/goal.urdf (robot description, URDF)
Before this commit: robot goal, 1 links, 0 joints
Links:
- link finish: geometry visual box size=1 3 0.05

File: Practica1/urdf_models/ramp.urdf (robot description, URDF)
Before this commit: robot ramp, 1 links, 0 joints
Links:
- removed link base
- added link block; visual box size=4 2 1.5
- added link rampa_bajada; visual box size=3.1 2 0.1
- added link rampa_subida; visual box size=3.1 2 0.1
Joints:
- added joint rampa_bajada_joint: type fixed, parent block, child rampa_bajada
- added joint rampa_subida_joint: type fixed, parent block, child rampa_subida
