Commit message: Add files via upload

File: Practica1/urdf_models/barrier.urdf (robot description, URDF)
Before this commit: robot barrier, 3 links, 2 joints
Links:
- link bar: mass None -> 5; geometry collision box size=0.1 2.22 0.2; visual box size=0.1 2.22 0.2
- link cylinder: mass None -> 10; geometry collision cylinder length=0.3 radius=0.2; visual cylinder length=0.3 radius=0.2
- link wrist_link: mass None -> 1; geometry collision cylinder length=0.2 radius=0.35; visual cylinder length=0.2 radius=0.35
Joints:
- joint rotation_joint: origin (none) -> xyz=0 0 0.5
- joint wrist_joint: origin xyz=0 0 -0.055 rpy=0 0 0 -> xyz=0 0.0 0.0

File: Practica1/urdf_models/ramp.urdf (robot description, URDF)
Before this commit: robot ramp, 3 links, 2 joints
Links:
- link block: mass None -> 10; geometry collision box size=4 2 1.5; visual box size=4 2 1.5
- link rampa_bajada: mass None -> 5; geometry collision box size=3.1 2 0.1; visual box size=3.1 2 0.1
- link rampa_subida: mass None -> 5; geometry collision box size=3.1 2 0.1; visual box size=3.1 2 0.1
